File: Proyecto_Bioimpedancia/Proyecto_Bioimpedancia.sch (KiCad schematic (older format))
At the start: 55 parts, among them J1 Jumper_Calibration, J2 Jumper, J3 Jumper, J4 Jumper, P1 CONN_01X03, P2 CONN_01X02, P3 CONN_01X02, P4 CONN_01X02, P5 CONN_01X02, P6 CONN_01X02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

Commit message: Muescas para asegurar a la carcasa anexadas
Diseño Final Preliminar
Parts:
- removed C10, C15, C16: 0,1uF, Capacitors_SMD:C_0805_HandSoldering, symbol 0,1uF
- removed C11, C19: 10uF, Capacitors_SMD:C_0805_HandSoldering, symbol 10uF
- removed U5: ADP3303, Housings_SOIC:SOIC-8_3.9x4.9mm_Pitch1.27mm, symbol ADP3303
- added C10, C11: 1uF, Capacitors_SMD:C_0805_HandSoldering, symbol 1uF
- added C14: 1nF, Capacitors_SMD:C_1206_HandSoldering, symbol 1nF
- added P7: CONN_01X02, Socket_Strips:Socket_Strip_Straight_1x02_Pitch2.54mm, symbol CONN_01X02
- added R13: 10K, Resistors_SMD:R_0805_HandSoldering, symbol 10K
- added R14: 78,7K, Resistors_SMD:R_0805_HandSoldering, symbol 78,7K
- added R15: 140K, Resistors_SMD:R_0805_HandSoldering, symbol 140K
- added U5: ADP3334, Housings_SOIC:SOIC-8_3.9x4.9mm_Pitch1.27mm, symbol ADP3334
- U1: footprint (none) -> Housings_SOIC:SOIC-8_3.9x4.9mm_Pitch1.27mm
Connections:
- net 3V3: now also C11.1, C14.2, R15.2, U5.5 (OUT), U5.6 (OUT)
- net AGND: now also C10.2, C11.2, R13.1, R14.1, U5.1 (GND)
- net V_FUENTE: now also C10.1, P7.2 (P2), U5.3 (IN), U5.4 (IN)
- new net: C14.1, R14.2, R15.1, U5.7 (FB)
- new net D_REG: P7.1 (P1), R13.2, U5.2 (SD)
Other:
- moved on the sheet: D2, R12
