File: Proyecto_Bioimpedancia/Proyecto_Bioimpedancia.kicad_pcb (KiCad board)
At the start: 2 copper layers, 61.1 x 34.4 mm, 59 parts, among them J1 Jumper_Calibration, J2 Jumper, J3 Jumper, J4 Jumper, P1 CONN_01X03, P2 CONN_01X02, P3 CONN_01X02, P4 CONN_01X02, P5 CONN_01X02, P6 CONN_01X02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

Commit message: Ultima versión para impresión
Final
Parts:
- removed REF** (x2): MountingHole_2.2mm_M2_DIN965_Pad, Mounting_Holes:MountingHole_2.7mm_M2.5_DIN965_Pad
Other:
- board size 61.1 x 34.4 mm -> 61.1 x 35.4 mm
Changed lines of the file:
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@@
     (links 124)
     (no_connects 0)
-    (area 165.072814 51.359999 242.483768 88.10912)
+    (area 165.352214 51.359999 242.483768 88.10912)
     (thickness 1.6)
     (drawings 18)
     (tracks 590)
     (zones 0)
-    (modules 59)
+    (modules 57)
     (nets 35)
   )
@@
     (add_net "Net-(U5-Pad8)")
   )
-  (module Mounting_Holes:MountingHole_2.7mm_M2.5_DIN965_Pad (layer F.Cu)
-    (at 179.9336 82.5881)
-    (descr "Mounting Hole 2.7mm, M2.5, DIN965")
-    (tags "mounting hole 2.7mm m2.5 din965")
-    (fp_text reference REF** (at 5.1689 1.5494) (layer F.SilkS) hide
-      (effects (font (size 1 1) (thickness 0.15)))
-    )
-    (fp_text value MountingHole_2.2mm_M2_DIN965_Pad (at 0 3.35) (layer F.Fab)
-      (effects (font (size 1 1) (thickness 0.15)))
-    )
-    (fp_circle (center 0 0) (end 2.35 0) (layer Cmts.User) (width 0.15))
-    (fp_circle (center 0 0) (end 2.6 0) (layer F.CrtYd) (width 0.05))
-    (pad 1 thru_hole circle (at 0 0) (size 4.7 4.7) (drill 2.7) (layers *.Cu *.Mask))
-  )
   (module Housings_SSOP:SSOP-16_5.3x6.2mm_Pitch0.65mm (layer F.Cu)
     (at 212.3948 68.2752 270)
@@
     )
   )
-  (module Mounting_Holes:MountingHole_2.7mm_M2.5_DIN965_Pad (layer F.Cu)
-    (at 179.8193 54.7624)
-    (descr "Mounting Hole 2.7mm, M2.5, DIN965")
-    (tags "mounting hole 2.7mm m2.5 din965")
-    (fp_text reference REF** (at 5.3086 0.0254) (layer F.SilkS) hide
-      (effects (font (size 1 1) (thickness 0.15)))
-    )
-    (fp_text value MountingHole_2.2mm_M2_DIN965_Pad (at 0 3.35) (layer F.Fab)
-      (effects (font (size 1 1) (thickness 0.15)))
-    )
-    (fp_circle (center 0 0) (end 2.35 0) (layer Cmts.User) (width 0.15))
-    (fp_circle (center 0 0) (end 2.6 0) (layer F.CrtYd) (width 0.05))
-    (pad 1 thru_hole circle (at 0 0) (size 4.7 4.7) (drill 2.7) (layers *.Cu *.Mask))
-  )
-  (gr_line (start 176.1109 85.8139) (end 176.1109 51.435) (angle 90) (layer Edge.Cuts) (width 0.15))
-  (gr_line (start 176.1109 51.435) (end 237.236 51.435) (angle 90) (layer Edge.Cuts) (width 0.15))
-  (gr_line (start 237.236 85.8139) (end 176.1109 85.8139) (angle 90) (layer Edge.Cuts) (width 0.15))
-  (gr_line (start 237.236 51.435) (end 237.236 85.8139) (angle 90) (layer Edge.Cuts) (width 0.15))
+  (gr_line (start 176.1109 86.0425) (end 176.1109 50.6476) (angle 90) (layer Edge.Cuts) (width 0.15))
+  (gr_line (start 237.236 86.0425) (end 176.1109 86.0425) (angle 90) (layer Edge.Cuts) (width 0.15))
+  (gr_line (start 237.236 50.6476) (end 237.236 86.0425) (angle 90) (layer Edge.Cuts) (width 0.15))
+  (gr_line (start 176.1109 50.6476) (end 237.236 50.6476) (angle 90) (layer Edge.Cuts) (width 0.15))
   (gr_text "SBS\nModule : 003" (at 214.1474 54.0639) (layer F.SilkS)
     (effects (font (size 1 1) (thickness 0.2)))
@@
     (polygon
       (pts
-        (xy 237.1598 85.7377) (xy 176.1871 85.7377) (xy 176.1871 51.5112) (xy 237.1598 51.5112) (xy 237.1598 85.7377)
+        (xy 237.1598 85.9663) (xy 176.1871 85.9663) (xy 176.1871 50.7238) (xy 237.1598 50.7238) (xy 237.1598 85.9663)
       )
     )
@@
         (xy 206.7941 56.2737) (xy 200.1266 56.2737) (xy 200.1266 64.8462) (xy 189.4205 64.8462) (xy 189.4205 63.0301)
         (xy 182.753 63.0301) (xy 182.753 64.8843) (xy 178.1937 64.8843) (xy 178.1937 66.5734) (xy 176.1871 66.5734)
-        (xy 176.1871 51.5112) (xy 237.1598 51.5112) (xy 237.1598 53.6956)
+        (xy 176.1871 50.7238) (xy 237.1598 50.7238) (xy 237.1598 53.6956)
       )
     )
@@
         (xy 192.3669 71.7931) (xy 192.3669 75.2094) (xy 206.3115 75.2094) (xy 206.3115 80.8736) (xy 219.5703 80.8736)
         (xy 219.5703 84.8995) (xy 220.4339 84.8995) (xy 220.4339 82.931) (xy 225.9584 82.931) (xy 225.9584 72.1741)
-        (xy 236.8677 72.1741) (xy 236.8677 85.7377) (xy 176.1871 85.7377) (xy 176.1871 67.7672) (xy 180.7591 67.7672)
+        (xy 236.8677 72.1741) (xy 236.8677 85.9663) (xy 176.1871 85.9663) (xy 176.1871 67.7672) (xy 180.7591 67.7672)
         (xy 180.7591 71.5645)
       )
